File: 3phase-FOC.kicad_sch (KiCad schematic)
At the start: 60 parts, among them J1 Debug-pin, J2 USB_C_Receptacle_USB2.0_16P, J3 Hall sensors_out, J4 Hall sensors_in, SW1 Board ON/OFF, U1 RP2350A, U10 BSC016N06NSTATMA1, U11 BSC016N06NSTATMA1, U12 BSC016N06NSTATMA1, U13 BSC016N06NSTATMA1, U14 BSC016N06NSTATMA1, U15 BSC016N06NSTATMA1, U2 W25Q32JVSS, U3 DRV8353RSRGZR, U5 ADS7042xDCU, U6 TLV75533PDBV, U7 TLV75533PDBV, U8 ADS7042xDCU, U9 ADS7042xDCU, Y1 Crystal

Commit message: added ext vbat->5v and 5v->3.3v and 3.3v_ref
Parts:
- removed JP1, JP3: EN_ALWAYS_ON, symbol Jumper:SolderJumper_3_Open
- added C19, C20, C21: 1uf (cog), symbol Device:C
- added C22: 100nF, symbol Device:C
- added C23, C24: 22uF, symbol Device:C
- added C25: 10uF, symbol Device:C
- added C26: 0.1 uF, symbol Device:C
- added C27, C28, C33: 47uF, symbol Device:C
- added C29, C30, C31, C32: 2.2uF, symbol Device:C
- added C34: 47pF, symbol Device:C
- added C35: 4700pf, symbol Device:C
- added C36, C38: 1uF, symbol Device:C
- added C37: 0.47uF, symbol Device:C
- added D2: B560C-13-F (48v schottky?), symbol Device:D_Schottky
- added JP5, JP6: EN_ALWAYS_ON, symbol Jumper:SolderJumper_3_Open
- added L2: 4.7 uH, symbol Device:L
- added L3: 7.2 uH, symbol Device:L
- added R11: 243k, symbol Device:R
- added R19, R20: 10k, symbol Device:R
- added R21: 10.2k, symbol Device:R
- added R22: 16.9k, symbol Device:R
- added R5: 150, symbol Device:R
- added U16: TPS54560BDDA, Package_SO:Texas_R-PDSO-G8_EP2.95x4.9mm_Mask2.4x3.1mm_ThermalVias, symbol Regulator_Switching:TPS54560BDDA
- added U17: REF3030, Package_TO_SOT_SMD:SOT-23, symbol Reference_Voltage:REF3030
- added U18: TLV75533PDBV, Package_TO_SOT_SMD:SOT-23-5, symbol Regulator_Linear:TLV75533PDBV
- added U4: AP63205WU, Package_TO_SOT_SMD:TSOT-23-6, symbol Regulator_Switching:AP63205WU
- C10, C13, C14: value 650pf -> 680pf
- R10, R4: value 100 -> 150
- R12: value 100 -> 90.9k
- R13: value 10k -> 442k
- R17: value 10k -> 53.6k
Connections:
- net +3.3V: now also C36.1, U18.5 (OUT)
- net +BATT: now also R13.1, C25.1, C29.1, C30.1, C31.1, C32.1, U16.2 (VIN), U4.2 (EN), U4.3 (IN)
- net -BATT: now also R12.2, C19.1, C20.1, C21.1, C23.2, C24.2, C25.2, C27.2, C28.2, C29.2, C30.2, C31.2, C32.2, C33.2, C34.2, C35.2, C36.2, C37.1, C38.2, D2.2 (A), R11.2, R19.2, R20.2, R21.2, U16.7 (GND), U16.9 (GND), U17.3 (GND), U18.2 (GND), U4.4 (GND); no longer R13.2, R17.2
- net 3.3v ref: no longer C8.1, U3.26 (VREF), U5.7 (AVDD), U8.7 (AVDD), U9.7 (AVDD)
- net EN_ADC_1: now also JP6.1 (A)
- net EN_ADC_3: now also JP5.1 (A)
- net I_meas_A: now also R10.1; no longer R12.1
- net I_meas_B: now also R5.1; no longer R10.1
- net at U9.4 (~{CS}): now also JP6.2 (C)
- net at C14.1, U9.6 (AINP): now also R10.2; no longer R12.2
- net at C13.1, U8.6 (AINP): now also R5.2; no longer R10.2
- net at U8.4 (~{CS}): now also JP5.2 (C)
- net +5V: now reaches R17.1
- net +5V: now also C23.1, C24.1, C27.1, C28.1, C33.1, C37.2, C38.1, L2.2, L3.2, U17.1 (IN), U18.1 (IN), U18.3 (EN), U4.1 (FB)
- new net: R17.2, R21.1, U16.5 (FB)
- new net: JP6.3 (B), R20.1
- new net: C22.1, L2.1, U4.5 (SW)
- new net: C22.2, U4.6 (BST)
- new net: C26.1, U16.1 (BOOT)
- new net: C26.2, D2.1 (K), L3.1, U16.8 (SW)
- new net: R11.1, R12.1, R13.2, U16.3 (EN), U16.4 (RT/CLK)
- new net: JP5.3 (B), R19.1
- new net: C35.1, R22.2
- new net 3.3V_VREF: C19.2, C20.2, C21.2, C8.1, U17.2 (OUT), U3.26 (VREF), U5.7 (AVDD), U8.7 (AVDD), U9.7 (AVDD)
- new net COMB: C34.1, R22.1, U16.6 (COMP)
Other:
- note added: "5v -> 3.3v and 3.3v_ref"
- note added: "Can probably replace the 4*C or 3*C with single/double C"
- note added: "Diodes corp - 0.6A max"
- note added: "TPS TI variant - 5A"
- note added: "VBAT -> 5V conversion"
- moved on the sheet: JP4, R18, U6, U7

Commit message: remoed DRV8353 internal buck comps
Parts:
- removed C18: 4*4.7 mid maybe?, symbol Device:C
- removed U6, U7: TLV75533PDBV, Package_TO_SOT_SMD:SOT-23-5, symbol Regulator_Linear:TLV75533PDBV
- added J5: Motor connector, symbol Connector:Screw_Terminal_01x03
- added J6: Bat connector, symbol Connector:Screw_Terminal_01x02
- added J7: HALL_3, symbol Connector:Conn_01x03_Pin
- added JP1: bulk-off, Jumper:SolderJumper-2_P1.3mm_Bridged_RoundedPad1.0x1.5mm, symbol Jumper:SolderJumper_2_Bridged
- added JP3: no-buck-pullup, symbol Jumper:SolderJumper_2_Bridged
- C11, C12, C7, D1, L1, R3, R6, R7, R8, R9, SW1: now not fitted
- C5: value V_in rated -> 1 uF; now not fitted
- C8: value 1uF -> 0.1uF
- J3: value Hall sensors_out -> HALL_1
- J4: value Hall sensors_in -> HALL_2
- R14, R15, R16: value 1mOhm -> 0.5mOhm
Connections:
- net -BATT is gone; now on net GND: C10.2, C12.2, C13.2, C14.2, C15.2, C16.1, C17.1, C19.1, C20.1, C21.1, C23.2, C24.2, C25.2, C27.2, C28.2, C29.2, C3.1, C30.2, C31.2, C32.2, C33.2, C34.2, C35.2, C36.2, C37.1, C38.2, C4.1, C5.1, C6.1, C7.2, C8.2, C9.2, D1.2 (A), D2.2 (A), R11.2, R12.2, R14.2, R15.2, R16.2, R18.2, R19.2, R20.2, R21.2, R6.2, R8.2, U16.7 (GND), U16.9 (GND), U17.3 (GND), U18.2 (GND), U3.1 (PGND), U3.12 (SNA), U3.13 (SNB), U3.22 (SNC), U3.27 (AGND), U3.41 (DGND), U3.49 (PAD), U4.4 (GND), U5.5 (AINM), U5.8 (GND), U8.5 (AINM), U8.8 (GND), U9.5 (AINM), U9.8 (GND)
- net +5V: now also J3.2 (Pin_2), J4.2 (Pin_2), J7.2 (Pin_2), JP3.1 (A)
- net +BATT: now also J6.1 (Pin_1)
- net LMOS_B: now also R15.1, U3.14 (SPB)
- net LMOS_C: now also R16.1, U3.21 (SPC)
- net Phase A: now also J5.1 (Pin_1)
- net Phase B: now also J5.2 (Pin_2)
- net Phase C: now also J5.3 (Pin_3)
- net nFault_DRV: no longer R2.2
- net at R3.1, U3.47 (RT_SD): now also JP1.1 (A)
- net at C7.1, R1.1, U3.44 (VCC): now also R2.2, JP3.2 (B)
- net GND: now reaches J4.1 (Pin_1)
- net GND: now also J3.1 (Pin_1), J6.2 (Pin_2), J7.1 (Pin_1), JP1.2 (B)
- net HALL_OUT_2: now reaches J4.3 (Pin_3)
- net HALL_OUT_1: now reaches J3.3 (Pin_3)
- new net HALL_OUT_3: J7.3 (Pin_3)
Other:
- note added: "- voltage refernce for the 3.3 ref X - better decoupling around ADCs for ref and PSU X - seperate ADC clocks (jumpers) X - ADC chip enables route to chip (with jumpters) X - make schematic look nicer - add more bypass capacitors (LDOs and MORE!) X - consider extra converter X - shunt ~1W max -> variable gain and solder in the relevant shunt resistance - lower shunt ref voltage - 3 vs 6 pwm? (i th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"
- note removed: "- voltage refernce for the 3.3 ref - better decoupling around ADCs for ref and PSU - seperate ADC clocks (jumpers) X - ADC chip enables route to chip (with jumpters) X - make schematic look nicer - add more bypass capacitors (LDOs and MORE!) - consider extra converter - shunt ~1W max -> variable gain and solder in the relevant shunt resistance - lower shunt ref voltage - 3 vs 6 pwm? (i thikn 3?) X"
- note removed: "LOD 3.3v stabilizers"
- note removed: "TLV76701DRVT instead? better PSSR"
- moved on the sheet: C10, C13, C14, C19, C20, C21, C9, J1, J2, J3, JP2, JP4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

Commit message: rpi harness
Parts:
- added C18, C39, C40: 4.7uF, symbol Device:C
- added C41, C44, C45, C46, C47, C48, C49, C50, C51, C52, C53: 100nF, symbol Device:C
- added C42, C43: 15pF, symbol Device:C
- added D3: D_Schottky, symbol Device:D_Schottky
- added JP7: WORSE_REF, symbol Jumper:SolderJumper_2_Bridged
- added JP8: BETTER_REF, symbol Jumper:SolderJumper_2_Open
- added L4: 3.3uH, AOTA-B201610S3R3-101-T:AOTA-B201610S3R3-101-T, symbol Device:L
- added R23: 33, symbol Device:R
- added R24, R27: 0, symbol Device:R
- added R25, R30, R33: 1k, symbol Device:R
- added R26: 10k, symbol Device:R
- added R28, R29: 5.1k, symbol Device:R
- added R31, R32: 27, symbol Device:R
- added SW2: BOOTSEL, Button_Switch_SMD:SW_SPST_B3U-1000P, symbol Switch:SW_Push
- added SW3: RPI_RST, Button_Switch_SMD:SW_SPST_B3U-1000P, symbol Switch:SW_Push
- U3: footprint RGZ0048L -> DRV8353FHRTAR:RGZ0048L
Connections:
- net +3.3V: now also U1.1 (IOVDD), U1.11 (IOVDD), U1.20 (IOVDD), U1.23 (DVDD), U1.30 (IOVDD), U1.38 (IOVDD), U1.39 (DVDD), U1.45 (IOVDD), U1.49 (VREG_VIN), U1.53 (USB_OTP_VDD), U1.54 (QSPI_IOVDD), U1.6 (DVDD), U2.8 (VCC), C39.1, C41.2, C44.1, C45.1, C46.1, C47.1, C48.1, C49.1, C50.1, JP7.2 (B), R23.1, R26.1
- net +5V: now also D3.1 (K)
- net 3.3V_VREF: now also JP8.1 (A)
- net GND: now also J1.3 (Pin_3), J2.A1 (GND), J2.A12 (GND), J2.B1 (GND), J2.B12 (GND), J2.SH (SHIELD), U1.47 (VREG_PGND), U1.61 (GND), U2.4 (GND), C18.2, C39.2, C40.2, C41.1, C42.1, C43.1, C44.2, C45.2, C46.2, C47.2, C48.2, C49.2, C50.2, C51.2, C52.2, C53.2, R28.1, R29.1, R33.2, SW2.1
- net MCU_TO_DRIVE_H_A: now also U1.9 (GPIO6)
- net MCU_TO_DRIVE_H_B: now also U1.10 (GPIO7)
- net MCU_TO_DRIVE_H_C: now also U1.12 (GPIO8)
- net VBUS: now reaches J2.A4 (VBUS), J2.A9 (VBUS), J2.B4 (VBUS), J2.B9 (VBUS)
- net VBUS: now also D3.2 (A)
- net at J2.A5 (CC1): now also R29.2
- net at J2.A6 (D+): now also J2.B6 (D+), R31.1
- net at J2.A7 (D-): now also J2.B7 (D-), R32.1
- net at J2.B5 (CC2): now also R28.2
- net GPIO_00_CS: now reaches U1.2 (GPIO0)
- net GPIO_00_CS: now also R27.1
- net X_IN: now reaches U1.21 (XIN)
- net X_IN: now also Y1.2, C42.2
- net X_OUT: now reaches U1.22 (XOUT)
- net X_OUT: now also R30.2
- net RUN: now reaches U1.26 (RUN)
- net RUN: now also SW3.1
- net RPI_ADC_REF: now reaches U1.44 (ADC_AVDD)
- net RPI_ADC_REF: now also JP7.1 (A), JP8.2 (B)
- net at U1.46 (VREG_AVDD): now also C40.1, R23.2
- net at U1.48 (VREG_LX): now also L4.2
- net +1.1V: now reaches U1.50 (VREG_FB)
- net +1.1V: now also C18.1, C51.1, C52.1, C53.1, L4.1
- net USB_DM: now reaches U1.51 (USB_DM)
- net USB_DM: now also R32.2
- net USB_DP: now reaches U1.52 (USB_DP)
- net USB_DP: now also R31.2
- net at U1.55 (QSPI_SD3): now also U2.7 (~{HOLD}/~{RESET}/IO_{3})
- net at U1.56 (QSPI_SCLK): now also U2.6 (CLK)
- net at U1.57 (QSPI_SD0): now also U2.5 (DI/IO_{0})
- net at U1.58 (QSPI_SD2): now also U2.3 (~{WP}/IO_{2})
- net at U1.59 (QSPI_SD1): now also U2.2 (DO/IO_{1})
- net at U1.60 (~{QSPI_SS}): now also R24.2, R25.1, R26.2, R27.2
- net at U2.1 (~{CS}): now also R24.1
- net at Y1.1: now also C43.2, R30.1
- new net: R33.1, SW3.2
- new net: R25.2, SW2.2
- no-connect marks 3 -> 5
Other:
- note added: "RPI2350 Decoupling"
- note removed: "2x 5.1k resistors to ground from CCx pins"
- moved on the sheet: C9, J6, U2, Y1

Commit message: bugfixes
Parts:
- removed C17: small and fast, symbol Device:C
- added C54, C55, C56, C57, C59, C60: 2.2uF, symbol Device:C
- added C58: 100nF, symbol Device:C
- C15, C16: value small and fast -> 100nF
- C26, C27, C28, C29, C30, C31, C32, C33, C34, C35, D2, L3, R11, R12, R13, R17, R21, R22, U16: now not fitted
- U17: value REF3030 -> REF3033
Connections:
- net MCU_TO_DRIVE_L_A is gone; now on net +5V: U3.35 (INLA)
- net MCU_TO_DRIVE_L_B is gone; now on net +5V: U3.37 (INLB)
- net MCU_TO_DRIVE_L_C is gone; now on net +5V: U3.39 (INLC)
- net +1.1V: now also U1.23 (DVDD), U1.39 (DVDD), U1.6 (DVDD)
- net +3.3V: no longer U1.23 (DVDD), U1.39 (DVDD), U1.6 (DVDD)
- net +5V: now also J3.3 (Pin_3), J4.3 (Pin_3), J7.3 (Pin_3); no longer J3.2 (Pin_2), J4.2 (Pin_2), J7.2 (Pin_2)
- net +BATT: now also C54.1, C55.1, C56.1, C57.1, C58.1, C59.2, C60.2
- net ADC_A_OUT: now also U1.16 (GPIO12)
- net ADC_B_OUT: now also U1.17 (GPIO13)
- net ADC_C_OUT: now also U1.18 (GPIO14)
- net ADC_clk_1: now also U1.19 (GPIO15)
- net ADC_clk_2: now also U1.27 (GPIO16)
- net ADC_clk_3: now also U1.28 (GPIO17)
- net EN_ADC_1: now also U1.13 (GPIO9)
- net EN_ADC_2: now also U1.14 (GPIO10)
- net EN_ADC_3: now also U1.15 (GPIO11)
- net GND: now also C54.2, C55.2, C56.2, C57.2, C58.2, C59.1, C60.1
- net HALL_OUT_1: now also J3.2 (Pin_2), U1.33 (GPIO21); no longer J3.3 (Pin_3)
- net HALL_OUT_2: now also J4.2 (Pin_2), U1.34 (GPIO22); no longer J4.3 (Pin_3)
- net HALL_OUT_3: now also J7.2 (Pin_2), U1.35 (GPIO23); no longer J7.3 (Pin_3)
- net at R12.1, R13.2, U16.3 (EN): no longer R11.1, U16.4 (RT/CLK)
- new net: R11.1, U16.4 (RT/CLK)
Other:
- note added: "3-pin PWM"
- note removed: "- voltage refernce for the 3.3 ref X - better decoupling around ADCs for ref and PSU X - seperate ADC clocks (jumpers) X - ADC chip enables route to chip (with jumpters) X - make schematic look nicer - add more bypass capacitors (LDOs and MORE!) X - consider extra converter X - shunt ~1W max -> variable gain and solder in the relevant shunt resistance - lower shunt ref voltage - 3 vs 6 pwm? (i th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"
- moved on the sheet: C42, C43, R30, R33, SW3, U14, U15, Y1

Commit message: bugfixes, prettyfing
Parts:
- removed JP3: no-buck-pullup, symbol Jumper:SolderJumper_2_Bridged
- removed JP4, JP5, JP6: EN_ALWAYS_ON, symbol Jumper:SolderJumper_3_Open
- added JP3: HALL_PWR_SLCT, symbol Jumper:SolderJumper_3_Open
- D1: value D_Shockley 60v 1A -> D_Schottky 60v 1A
- R18, R19, R20: value 10k -> 4.7k
Connections:
- net +3.3V: now also R1.1, R2.2, U3.35 (INLA), U3.37 (INLB), U3.39 (INLC), JP3.1 (A)
- net +5V: now also JP3.3 (B); no longer J3.3 (Pin_3), J4.3 (Pin_3), J7.3 (Pin_3), U3.35 (INLA), U3.37 (INLB), U3.39 (INLC)
- net EN_ADC_1: now also U9.4 (~{CS})
- net EN_ADC_2: now also U8.4 (~{CS})
- net EN_ADC_3: now also U5.4 (~{CS})
- net GND: no longer R18.2, R19.2, R20.2
- net HALL_OUT_1: now also R20.1
- net HALL_OUT_2: now also R19.1
- net HALL_OUT_3: now also R18.1
- net at C7.1, U3.44 (VCC): no longer R1.1, R2.2
- new net HALL_PWR: J3.3 (Pin_3), J4.3 (Pin_3), J7.3 (Pin_3), JP3.2 (C), R18.2, R19.2, R20.2
Other:
- note added: "Diodes corp - 0.6A and 32V max"
- note added: "HALL SENSORS"
- note added: "Power IO"
- note added: "RPI - RST, ADC_REF, Crystal"
- note added: "USB-RPI"
- note removed: "Diodes corp - 0.6A max"
- moved on the sheet: C1, C10, C11, C12, C13, C14, C15, C16, C18, C19, C2, C20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

Commit message: final v0
Parts:
- removed C16: 100nF, symbol Device:C
- removed D1: D_Schottky 60v 1A, symbol Device:D_Shockley
- added C17, C61, C62, C63: 470uF, symbol Device:C
- added C64: 100nF, symbol Device:C
- added C65, C66, C67: 4.7uF, symbol Device:C
- added D1: D_Schottky - 60v, symbol Device:D_Schottky
- added D4: D_Schottky 3v, symbol Device:D_Schottky
- added J8: UNUSED_ADC, symbol Connector:Conn_01x03_Pin
- added J9: UNUSED_GPIO, symbol Connector:Conn_01x04_Pin
- added JP4: 3_PIN_HD_SF, symbol Jumper:SolderJumper_3_Open
- added R34: 100k, symbol Device:R
- added R35: 4.7k, symbol Device:R
- C54, C55, C56, C57, C59, C60: value 2.2uF -> 4.7uF
- C9: value >10uF -> 10nF; now not fitted
Connections:
- net +3.3V: now also R1.2, R18.1, R19.1, R20.1, JP4.3 (B); no longer R1.1, U3.35 (INLA), U3.37 (INLB), U3.39 (INLC)
- net +BATT: now also C59.1, C60.1, C17.1, C61.1, C62.1, C63.1, C64.1, C65.1, C66.1, C67.1, R34.1; no longer C59.2, C60.2, C9.1
- net GND: now also C59.2, C60.2, C17.2, C61.2, C62.2, C63.2, C64.2, C65.2, C66.2, C67.2, D1.2 (A), D4.2 (A), R35.2; no longer C59.1, C60.1
- net GPIO_00_CS: now also J9.1 (Pin_1)
- net HALL_OUT_1: now also R20.2; no longer R20.1
- net HALL_OUT_2: now also R19.2; no longer R19.1
- net HALL_OUT_3: now also R18.2; no longer R18.1
- net HALL_PWR: no longer R18.2, R19.2, R20.2
- net nFault_DRV: now also R1.1; no longer R1.2
- net UN_GPIO_18: now reaches U1.29 (GPIO18)
- net UN_GPIO_18: now also J9.3 (Pin_3)
- net UN_GPIO_01: now reaches U1.3 (GPIO1)
- net UN_GPIO_01: now also J9.2 (Pin_2)
- net UN_GPIO_19: now reaches U1.31 (GPIO19)
- net UN_GPIO_19: now also J9.4 (Pin_4)
- net SET_3_PINMODE: now reaches U1.32 (GPIO20)
- net SET_3_PINMODE: now also JP4.1 (A)
- net at U1.40 (GPIO26/ADC0): now also C9.1, D4.1 (K), R34.2, R35.1
- net at U1.41 (GPIO27/ADC1): now also J8.1 (Pin_1)
- net at U1.42 (GPIO28/ADC2): now also J8.2 (Pin_2)
- net at U1.43 (GPIO29/ADC3): now also J8.3 (Pin_3)
- net at C11.2, L1.2, U3.42 (SW): now also D1.1 (K)
- new net MCU_TO_DRIVE_L_A: JP4.2 (C), U3.35 (INLA), U3.37 (INLB), U3.39 (INLC)
Other:
- note added: "Bulk bat supply"
- moved on the sheet: C11, C12, C15, C18, C40, C54, C55, C56, C57, C58, JP1, L1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

Commit message: adding footprints
Parts:
- removed D4: D_Schottky 3v, symbol Device:D_Schottky
- removed JP4: 3_PIN_HD_SF, symbol Jumper:SolderJumper_3_Open
- added C1, C15, C25: 1uf, symbol Device:C
- added C20, C28, C3: 100nf, symbol Device:C
- added D3: PDZ3.0B,115, Diode_SMD:D_SOD-323_HandSoldering, symbol Device:D_Zener
- added JP2: 3_PIN_HD_SF, Jumper:SolderJumper-3_P1.3mm_Bridged12_RoundedPad1.0x1.5mm, symbol Jumper:SolderJumper_3_Bridged12
- C19: renamed from C20; value 1uf (cog) -> 100nF c0g
- C2: renamed from C21; value 1uf (cog) -> 100nf (cog)
- C27: renamed from C19; value 1uf (cog) -> 100nf c0g
- D4: renamed from D3; value D_Schottky -> 1N4148W-7-F; footprint (none) -> Diode_SMD:Nexperia_CFP3_SOD-123W
- J2: renamed from J8; footprint (none) -> Connector_PinHeader_2.54mm:PinHeader_1x03_P2.54mm_Vertical
- J4: renamed from J9; footprint (none) -> Connector_PinSocket_2.54mm:PinSocket_1x04_P2.54mm_Vertical
- J5: footprint (none) -> Connector_PinHeader_2.54mm:PinHeader_1x03_P2.54mm_Vertical
- J7: footprint (none) -> Connector_PinSocket_2.54mm:PinSocket_1x03_P2.54mm_Vertical
- J8: renamed from J4; footprint (none) -> Connector_PinSocket_2.54mm:PinSocket_1x03_P2.54mm_Vertical
- J9: renamed from J3; footprint (none) -> Connector_PinSocket_2.54mm:PinSocket_1x03_P2.54mm_Vertical
- JP1: renamed from JP2; footprint (none) -> Jumper:SolderJumper-3_P1.3mm_Open_RoundedPad1.0x1.5mm
- JP4: renamed from JP3; footprint (none) -> Jumper:SolderJumper-3_P1.3mm_Open_RoundedPad1.0x1.5mm
- JP5: renamed from JP7; footprint (none) -> Jumper:SolderJumper-2_P1.3mm_Bridged2Bar_RoundedPad1.0x1.5mm
- JP6: renamed from JP8; footprint (none) -> Jumper:SolderJumper-2_P1.3mm_Open_RoundedPad1.0x1.5mm
- R1: renamed from R10; footprint (none) -> Resistor_SMD:R_0603_1608Metric_Pad0.98x0.95mm_HandSolder
- R10: renamed from R23; footprint (none) -> Resistor_SMD:R_0603_1608Metric_Pad0.98x0.95mm_HandSolder
- R11: renamed from R2; footprint (none) -> Resistor_SMD:R_0603_1608Metric_Pad0.98x0.95mm_HandSolder
- R13: renamed from R1; footprint (none) -> Resistor_SMD:R_0603_1608Metric_Pad0.98x0.95mm_HandSolder
- R15: renamed from R25; footprint (none) -> Resistor_SMD:R_0603_1608Metric_Pad0.98x0.95mm_HandSolder
- R16: renamed from R26; footprint (none) -> Resistor_SMD:R_0603_1608Metric_Pad0.98x0.95mm_HandSolder
- R17: renamed from R27; footprint (none) -> Resistor_SMD:R_0603_1608Metric_Pad0.98x0.95mm_HandSolder
- R19: renamed from R24; footprint (none) -> Resistor_SMD:R_0603_1608Metric_Pad0.98x0.95mm_HandSolder
- R2: renamed from R22; footprint (none) -> Resistor_SMD:R_0603_1608Metric_Pad0.98x0.95mm_HandSolder
- R20: renamed from R7; footprint (none) -> Resistor_SMD:R_0603_1608Metric_Pad0.98x0.95mm_HandSolder
- R21: renamed from R9; footprint (none) -> Resistor_SMD:R_0603_1608Metric_Pad0.98x0.95mm_HandSolder
- R22: renamed from R8; footprint (none) -> Resistor_SMD:R_0603_1608Metric_Pad0.98x0.95mm_HandSolder
- R23: renamed from R34; footprint (none) -> Resistor_SMD:R_0603_1608Metric_Pad0.98x0.95mm_HandSolder
- R24: renamed from R6; footprint (none) -> Resistor_SMD:R_0603_1608Metric_Pad0.98x0.95mm_HandSolder
- R25: renamed from R35; footprint (none) -> Resistor_SMD:R_0603_1608Metric_Pad0.98x0.95mm_HandSolder
- R26: renamed from R3; footprint (none) -> Resistor_SMD:R_0603_1608Metric_Pad0.98x0.95mm_HandSolder
- R27: renamed from R18; footprint (none) -> Resistor_SMD:R_0603_1608Metric_Pad0.98x0.95mm_HandSolder
- R28: renamed from R19; footprint (none) -> Resistor_SMD:R_0603_1608Metric_Pad0.98x0.95mm_HandSolder
- R29: renamed from R20; footprint (none) -> Resistor_SMD:R_0603_1608Metric_Pad0.98x0.95mm_HandSolder
- R3: renamed from R13; footprint (none) -> Resistor_SMD:R_0603_1608Metric_Pad0.98x0.95mm_HandSolder
- R30: renamed from R33; footprint (none) -> Resistor_SMD:R_0603_1608Metric_Pad0.98x0.95mm_HandSolder
- R31: renamed from R28; footprint (none) -> Resistor_SMD:R_0603_1608Metric_Pad0.98x0.95mm_HandSolder
- R32: renamed from R29; footprint (none) -> Resistor_SMD:R_0603_1608Metric_Pad0.98x0.95mm_HandSolder
- R33: renamed from R30; footprint (none) -> Resistor_SMD:R_0603_1608Metric_Pad0.98x0.95mm_HandSolder
- R34: renamed from R31; footprint (none) -> Resistor_SMD:R_0603_1608Metric_Pad0.98x0.95mm_HandSolder
- R35: renamed from R32; footprint (none) -> Resistor_SMD:R_0603_1608Metric_Pad0.98x0.95mm_HandSolder
- R4: renamed from R17; footprint (none) -> Resistor_SMD:R_0603_1608Metric_Pad0.98x0.95mm_HandSolder
- R5: renamed from R21; footprint (none) -> Resistor_SMD:R_0603_1608Metric_Pad0.98x0.95mm_HandSolder
- R6: renamed from R12; footprint (none) -> Resistor_SMD:R_0603_1608Metric_Pad0.98x0.95mm_HandSolder
- R7: renamed from R11; footprint (none) -> Resistor_SMD:R_0603_1608Metric_Pad0.98x0.95mm_HandSolder
- R8: renamed from R5; footprint (none) -> Resistor_SMD:R_0603_1608Metric_Pad0.98x0.95mm_HandSolder
- R9: renamed from R4; footprint (none) -> Resistor_SMD:R_0603_1608Metric_Pad0.98x0.95mm_HandSolder
- U10: renamed from U13; footprint TDSON-8_INF -> BSC016N06NS:TDSON-8_INF
- U11: footprint TDSON-8_INF -> BSC016N06NS:TDSON-8_INF
- U12: renamed from U14; footprint TDSON-8_INF -> BSC016N06NS:TDSON-8_INF
- U13: renamed from U15; footprint TDSON-8_INF -> BSC016N06NS:TDSON-8_INF
- U8: renamed from U12; footprint TDSON-8_INF -> BSC016N06NS:TDSON-8_INF
- U9: renamed from U10; footprint TDSON-8_INF -> BSC016N06NS:TDSON-8_INF
- renumbered C26 to C10, C32 to C11, C31 to C12, C30 to C13, C29 to C14, C27 to C16, C28 to C17, C33 to C18, C13 to C21, C25 to C26, C10 to C29, C67 to C30, C55 to C31, C54 to C32, C66 to C33, C15 to C34, C44 to C35, C45 to C36, C46 to C37, C47 to C38, C48 to C39, C37 to C4, C49 to C40, C50 to C41, C56 to C42, C3 to C43, C2 to C44, C57 to C45, C51 to C46, C52 to C47, C53 to C48, C1 to C49, C34 to C5, C58 to C50, C65 to C51, C6 to C52, C59 to C53, C60 to C54, C64 to C55, C39 to C56, C18 to C57, C40 to C58, C41 to C59, C38 to C6, C8 to C60, C5 to C61, C4 to C62, C11 to C63, C7 to C64, C12 to C65, C9 to C66, C42 to C67, C43 to C68, C17 to C69, C36 to C7, C61 to C70, C62 to C71, C63 to C72, C14 to C8, C35 to C9, D2 to D1, D1 to D2, J6 to J3, J2 to J6, JP1 to JP3, L3 to L1, L4 to L3, L1 to L4, R16 to R12, R15 to R14, R14 to R18, SW2 to SW1, SW1 to SW2, U17 to U1, U3 to U14, U1 to U15, U2 to U16, U9 to U2, U18 to U3, U16 to U4, U8 to U5, U4 to U6, U5 to U7
Connections:
- net +3.3V: now also C20.1, C28.1, C3.1, JP2.3 (B)
- net 3.3V_VREF: now also C1.2, C15.2, C25.2
- net GND: now also C1.1, C15.1, C20.2, C25.1, C28.2, C3.2, D3.2 (A)
- net MCU_TO_DRIVE_L_A: now also JP2.2 (C)
- net SET_3_PINMODE: now also JP2.1 (A)
- net at C66.1, R23.2, R25.1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: now also D3.1 (K)
Other:
- moved on the sheet: C19, C21, C27, C29, C46, C47, C48, R8, R9, U5, U7

Commit message: adding footprints
Parts:
- removed C69, C70: 470uF, symbol Device:C
- removed Y1: Crystal, symbol Device:Crystal
- added C73, C74: 470uF, Capacitor_THT:CP_Radial_D10.0mm_P5.00mm, symbol Device:C_Polarized
- added X1: ABM8-272-T3, ABM8-272-T3:ABM8-272-T3_ABR, symbol ABM8-272-T3:ABM8-272-T3
- C1, C15, C25: footprint (none) -> Capacitor_SMD:C_0603_1608Metric_Pad1.08x0.95mm_HandSolder
- C19, C2, C27: footprint (none) -> Resistor_SMD:R_1206_3216Metric_Pad1.30x1.75mm_HandSolder
- C20, C28, C3: footprint (none) -> Capacitor_SMD:C_0402_1005Metric_Pad0.74x0.62mm_HandSolder
- C71, C72: value 470uF -> 4.7uF; footprint (none) -> Capacitor_SMD:C_1206_3216Metric_Pad1.33x1.80mm_HandSolder
- D1, D2: footprint (none) -> Diode_SMD:D_SMC_Handsoldering
- J6: footprint (none) -> Connector_USB:USB_C_Receptacle_Palconn_UTC16-G
- L1: value 7.2 uH -> 10 uH; footprint (none) -> Inductor_SMD:L_Bourns_SRR1208_12.7x12.7mm
- L2: footprint (none) -> Inductor_SMD:L_Bourns_SRP7028A_7.3x6.6mm
Connections:
- net +BATT: now also C73.1, C74.1
- net GND: now also C73.2, C74.2, X1.2, X1.4
- net X_IN: now also X1.1
- net at C68.2, R33.1: now also X1.3
Other:
- note added: "VBAT SENS"
- moved on the sheet: C66, C67, C68, D3, JP5, JP6, R1, R23, R25, R30, R33, R8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
