File: 3phase-FOC.kicad_sch (KiCad schematic)
At the start: 150 parts, among them J1 Debug-pin, J2 UNUSED_ADC, J3 Bat connector, J4 UNUSED_GPIO, J5 Motor connector, J6 USB_C_Receptacle_USB2.0_16P, J7 HALL_3, J8 HALL_2, J9 HALL_1, SW1 BOOTSEL, SW2 Board ON/OFF, SW3 RPI_RST, U1 REF3033, U10 BSC016N06NSTATMA1, U11 BSC016N06NSTATMA1, U12 BSC016N06NSTATMA1, U13 BSC016N06NSTATMA1, U14 DRV8353RSRGZR, U15 RP2350A, U16 W25Q32JVSS, U2 ADS7042xDCU, U3 TLV75533PDBV, U4 TPS54560BDDA, U5 ADS7042xDCU, U6 AP63205WU, U7 ADS7042xDCU, U8 BSC016N06NSTATMA1, U9 BSC016N06NSTATMA1, X1 ABM8-272-T3

Commit message: finishing footprints and switch lib
Parts:
- C10, C11, C12, C13, C14, C16, C17, C18, C21, C22, C23, C24, C29, C34, C4, C43, C44, C49, C5, C50, C52, C55, C56, C57, C58, C59, C6, C60, C61, C62, C63, C64, C66, C67, C68, C7, C8, C9, J3: footprint (none) -> Capacitor_SMD:C_0603_1608Metric_Pad1.08x0.95mm_HandSolder
- C26, C30, C31, C32, C33, C42, C45, C51, C53, C54: footprint (none) -> Capacitor_SMD:C_1206_3216Metric_Pad1.33x1.80mm_HandSolder
- C35, C36, C37, C38, C39, C40, C41, C46, C47, C48: footprint (none) -> Capacitor_SMD:C_0402_1005Metric_Pad0.74x0.62mm_HandSolder
- C65: footprint (none) -> Capacitor_SMD:C_0805_2012Metric_Pad1.18x1.45mm_HandSolder
- SW2: footprint (none) -> Button_Switch_THT:SW_DIP_SPSTx03_Slide_9.78x9.8mm_W7.62mm_P2.54mm

Commit message: footprint done, final schema changes done
Parts:
- J3: footprint Capacitor_SMD:C_0603_1608Metric_Pad1.08x0.95mm_HandSolder -> Connector_AMASS:AMASS_XT90PW-M_1x02_P10.90mm_Horizontal
- J5: footprint Connector_PinHeader_2.54mm:PinHeader_1x03_P2.54mm_Vertical -> Connector_Wire:SolderWire-6sqmm_1x03_P14mm_D3.5mm_OD7mm
- L4: footprint (none) -> Inductor_SMD:L_12x12mm_H6mm
- R12, R14, R18: footprint (none) -> Resistor_SMD:R_2512_6332Metric_Pad1.40x3.35mm_HandSolder
- R21: value 2 ohm -> 3 ohm
- SW2: footprint Button_Switch_THT:SW_DIP_SPSTx03_Slide_9.78x9.8mm_W7.62mm_P2.54mm -> switch:SHOU HAN MST-22D18G2 3J
Other:
- moved on the sheet: C10, C11, C12, C13, C14, C16, C17, C18, C22, C23, C24, C26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
